File: modulogue_vco.kicad_sch (KiCad schematic)
At the start: 107 parts, among them J1 SAWTOOTH, J2 TRIANGLE, J3 AudioJack2, J4 AudioJack2, J5 AudioJack2, J6 NOISE, J7 HP NOISE, J8 CV IN, Q2 2N3904, Q3 2N5457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

Commit message: update pulse
Parts:
- added C33: 47uF, symbol Device:C_Polarized
- added D10: POWER ON, symbol Device:LED
- added J10: CV IN, symbol Connector_Audio:AudioJack2_SwitchT
- added R35: 1K, symbol Device:R
- added R36: 10K, symbol Device:R_Trim
- J3: value AudioJack2 -> SINE
- J4: value AudioJack2 -> PULSE
- J5: value AudioJack2 -> MIX OUT
- J8: value CV IN -> LFO
- J9: value ~ -> Eurorack Power
Connections:
- net +5V: now also C33.1, D10.2 (A)
- net CV IN: no longer J8.T, U3.2 (B)
- net GND: now also C33.2, J10.S, R35.2
- net PIN +12V: no longer D9.2 (A)
- net PIN +5V: now also D9.2 (A)
- net PIN CV: now also J10.TN
- net at C1.1, Q2.3 (C), R1.1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: now also R36.2
- net at C1.2, RV1.3, U1.1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: now also R36.1
- net FILTERED NOISE: no longer names the net of R25.1, U10.3 (+), U5.7, U8.3 (+), U8.5 (+), U9.3 (+), U9.5 (+)
- net LFO: no longer names the net of R12.2
- net LFO: now also J8.T
- new net: D10.1 (K), R35.1
- new net: J10.T, U3.2 (B)
Other:
- moved on the sheet: C1, C10, C21, C8, C9, J1, J2, J3, J4, J5, J6, J7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

Commit message: update schematic layout
Parts:
- removed Q2: 2N3904, Package_TO_SOT_THT:TO-92_Inline, symbol Transistor_BJT:2N3904
- removed R3: 1K, symbol Device:R
- removed R36: 10K, symbol Device:R_Trim
- added Q1: 2N3904, Package_TO_SOT_THT:TO-92_Inline, symbol Transistor_BJT:2N3904
- added R3: 10K, symbol Device:R_Trim
- added R36: 10K, symbol Device:R
- C1: value 22nF -> 100nF
- C21: value 100nF -> 22nF
- R2: value 10K -> 1K
Connections:
- net +12V: now also C1.2, C2.1; no longer C2.2, C21.1
- net GND: now also C1.1, C2.2, R2.2, Q1.1 (E); no longer C2.1, C21.2
- net SAW: now also R36.2; no longer R2.2
- net at U3.3 (E): now also R2.1
- net at R1.1, RV1.2, U1.2 (-): now also C21.1, Q1.3 (C), R3.2; no longer C1.1
- net at RV1.3, U1.1, U2.1: now also C21.2, R3.1; no longer C1.2
- new net: Q1.2 (B), R36.1
Other:
- moved on the sheet: C10, C11, C12, C13, C14, C15, C16, C17, C18, C19, C20, C22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
